Commit message: docs(arm): 팔 관절 가동범위 실기 측정·확정값 반영
- arm.xacro: 관절별 limit을 측정값으로 (joint_limit 공통 ±π 제거, 매크로에 lower/upper 추가)
  joint1 ±175°, joint2 -95°..+113°, joint3 -111°..+82°, joint4 -99°..+117°, joint5_wrist_roll ±170°
- arm_params.yaml: motor_ids [11,12,13,14,16,15], joint_min_rad / joint_max_rad (그리퍼 -134°..-3° 포함)
- 출처: 2026-10-27 실기 보정 (OpenCR#2 nz2_arm_v2, 기계/케이블 끝에서 7° 안쪽)
- [가정] 모터 부호 +1 — URDF 축 방향과 실제 회전 방향 확인 필요
- joint4 접힘 인터락(+6.5°)은 정적 한계로 못 나타내 주석으로만 남김

Refs #19

File: ros2_ws/src/nz2_description/urdf/arm.xacro (robot description, xacro)
@@ -19,6 +19,8 @@
   <xacro:property name="wrist_length" value="0.0"/>   <!-- joint4 → 손목 롤 (TODO) -->
   <xacro:property name="gripper_length" value="0.0"/> <!-- 손목 롤 → 집게 끝 (TODO) -->
-  <xacro:property name="joint_limit" value="${pi}"/>  <!-- TODO: arm_params.yaml과 맞추기 -->
-  <xacro:macro name="arm_joint" params="name parent child xyz axis">
+  <!-- 관절 가동범위 [rad]: 2026-10-27 실기 측정·확정 (OpenCR#2 nz2_arm_v2, 기계/케이블 끝에서 7° 안쪽).
+       config/arm_params.yaml의 joint_min_rad / joint_max_rad와 같은 값.
+       [가정] 모터 부호 +1 기준. 실제 회전 방향이 URDF 축과 반대면 lower/upper를 부호 반전해 맞춘다 (확인 필요). -->
+  <xacro:macro name="arm_joint" params="name parent child xyz axis lower upper">
     <link name="${child}"/>
     <joint name="${name}" type="revolute">
@@ -27,5 +29,5 @@
       <origin xyz="${xyz}"/>
       <axis xyz="${axis}"/>
-      <limit lower="${-joint_limit}" upper="${joint_limit}" effort="1.0" velocity="1.0"/> <!-- TODO -->
+      <limit lower="${lower}" upper="${upper}" effort="1.0" velocity="1.0"/> <!-- effort·velocity TODO -->
     </joint>
   </xacro:macro>
@@ -37,10 +39,19 @@
       <origin xyz="${x} 0 ${z}"/>
     </joint>
-    <xacro:arm_joint name="joint1" parent="arm_base_link" child="arm_link1" xyz="0 0 0" axis="0 0 1"/>
-    <xacro:arm_joint name="joint2" parent="arm_link1" child="arm_link2" xyz="0 0 ${base_to_joint2}" axis="0 1 0"/>
-    <xacro:arm_joint name="joint3" parent="arm_link2" child="arm_link3" xyz="0 0 ${link1_length}" axis="0 1 0"/>
-    <xacro:arm_joint name="joint4" parent="arm_link3" child="arm_link4" xyz="${link2_length} 0 0" axis="0 1 0"/>
-    <!-- 손목 롤 (추가 관절): 집게 중심선 둘레 회전 -->
-    <xacro:arm_joint name="joint5_wrist_roll" parent="arm_link4" child="arm_link5" xyz="${wrist_length} 0 0" axis="1 0 0"/>
+    <!-- ID11 ±175° -->
+    <xacro:arm_joint name="joint1" parent="arm_base_link" child="arm_link1" xyz="0 0 0" axis="0 0 1"
+                     lower="-3.0543" upper="3.0543"/>
+    <!-- ID12 -95° .. +113° -->
+    <xacro:arm_joint name="joint2" parent="arm_link1" child="arm_link2" xyz="0 0 ${base_to_joint2}" axis="0 1 0"
+                     lower="-1.6581" upper="1.9722"/>
+    <!-- ID13 -111° .. +82° -->
+    <xacro:arm_joint name="joint3" parent="arm_link2" child="arm_link3" xyz="0 0 ${link1_length}" axis="0 1 0"
+                     lower="-1.9373" upper="1.4312"/>
+    <!-- ID14 -99° .. +117°. 접힌 자세에서는 +6.5°(0.1134 rad)까지만 (인터락) — 정적 한계로는 표현 못 해 펌웨어가 막는다 -->
+    <xacro:arm_joint name="joint4" parent="arm_link3" child="arm_link4" xyz="${link2_length} 0 0" axis="0 1 0"
+                     lower="-1.7279" upper="2.0420"/>
+    <!-- 손목 롤 (추가 관절): 집게 중심선 둘레 회전. ID16 ±170° -->
+    <xacro:arm_joint name="joint5_wrist_roll" parent="arm_link4" child="arm_link5" xyz="${wrist_length} 0 0" axis="1 0 0"
+                     lower="-2.9671" upper="2.9671"/>
     <link name="gripper_link"/>
     <joint name="gripper_joint" type="fixed">
